Commit message: Update sorobotics_dog.urdf

File: sorobotics_dog.urdf (robot description, URDF)
Before this commit: robot sorobotics_codenamedog_rviz, 23 links, 22 joints
Links:
- link base_link: geometry collision box size=0.14 0.11 0.07; visual mesh filename=package://sorobotics_codenamedog_mechanics/stl/mainbody.stl scale=0.001 0.001 0.001
- link front_left_foot_link: geometry collision box size=0.026 0.020 0.13; visual mesh filename=package://sorobotics_codenamedog_mechanics/stl/lfoot.stl scale=0.001 0.001 0.001
- link front_left_leg_link: geometry collision box size=0.028 0.036 0.1075; visual mesh filename=package://sorobotics_codenamedog_mechanics/stl/larm.stl scale=0.001 0.001 0.001
- link front_left_leg_link_cover: geometry visual mesh filename=package://sorobotics_codenamedog_mechanics/stl/larm_cover.s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 scale=0.001 0.001 0.001
- link front_left_shoulder_link: geometry collision box size=0.044 0.038 0.07; visual mesh filename=package://sorobotics_codenamedog_mechanics/stl/lshoulder.stl scale=0.001 0.001 0.001
- link front_left_toe_link: geometry collision sphere radius=0.02; visual mesh filename=package://sorobotics_codenamedog_mechanics/stl/foot.stl scale=0.001 0.001 0.001
- link front_link: geometry collision box size=0.058 0.11 0.07; visual mesh filename=package://sorobotics_codenamedog_mechanics/stl/frontpart.stl scale=0.001 0.001 0.001
- link front_right_foot_link: geometry collision box size=0.026 0.020 0.13; visual mesh filename=package://sorobotics_codenamedog_mechanics/stl/rfoot.stl scale=0.001 0.001 0.001
- link front_right_leg_link: geometry collision box size=0.028 0.036 0.1075; visual mesh filename=package://sorobotics_codenamedog_mechanics/stl/rarm.stl scale=0.001 0.001 0.001
- link front_right_leg_link_cover: geometry visual mesh filename=package://sorobotics_codenamedog_mechanics/stl/rarm_cover.s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 scale=0.001 0.001 0.001
- link front_right_shoulder_link: geometry collision box size=0.044 0.038 0.07; visual mesh filename=package://sorobotics_codenamedog_mechanics/stl/rshoulder.stl scale=0.001 0.001 0.001
- link front_right_toe_link: geometry collision sphere radius=0.02; visual mesh filename=package://sorobotics_codenamedog_mechanics/stl/foot.stl scale=0.001 0.001 0.001
- link rear_left_foot_link: geometry collision box size=0.026 0.020 0.13; visual mesh filename=package://sorobotics_codenamedog_mechanics/stl/lfoot.stl scale=0.001 0.001 0.001
- link rear_left_leg_link: geometry collision box size=0.028 0.036 0.1075; visual mesh filename=package://sorobotics_codenamedog_mechanics/stl/larm.stl scale=0.001 0.001 0.001
- link rear_left_leg_link_cover: geometry visual mesh filename=package://sorobotics_codenamedog_mechanics/stl/larm_cover.s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 scale=0.001 0.001 0.001
- link rear_left_shoulder_link: geometry collision box size=0.044 0.038 0.07; visual mesh filename=package://sorobotics_codenamedog_mechanics/stl/lshoulder.stl scale=0.001 0.001 0.001
- link rear_left_toe_link: geometry collision sphere radius=0.02; visual mesh filename=package://sorobotics_codenamedog_mechanics/stl/foot.stl scale=0.001 0.001 0.001
- link rear_link: geometry collision box size=0.04 0.11 0.07; visual mesh filename=package://sorobotics_codenamedog_mechanics/stl/backpart.stl scale=0.001 0.001 0.001
- link rear_right_foot_link: geometry collision box size=0.026 0.020 0.13; visual mesh filename=package://sorobotics_codenamedog_mechanics/stl/rfoot.stl scale=0.001 0.001 0.001
- link rear_right_leg_link: geometry collision box size=0.028 0.036 0.1075; visual mesh filename=package://sorobotics_codenamedog_mechanics/stl/rarm.stl scale=0.001 0.001 0.001
- link rear_right_leg_link_cover: geometry visual mesh filename=package://sorobotics_codenamedog_mechanics/stl/rarm_cover.s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 scale=0.001 0.001 0.001
- link rear_right_shoulder_link: geometry collision box size=0.044 0.038 0.07; visual mesh filename=package://sorobotics_codenamedog_mechanics/stl/rshoulder.stl scale=0.001 0.001 0.001
- link rear_right_toe_link: geometry collision sphere radius=0.02; visual mesh filename=package://sorobotics_codenamedog_mechanics/stl/foot.stl scale=0.001 0.001 0.001
